File: hw/kegboard-coaster-alt/kegboard-coaster-alt.brd (EAGLE design)
At the start: 44.5 x 25.4 mm, 11 parts

Commit message: Update coaster to v2.1.
Routing:
- net ONEWIRE_B: track 25.4 -> 44.4 mm, vias 1 -> 0
- net GND: track 102.3 -> 105.8 mm
- net GPIO_B: track 23.1 -> 26.1 mm
- net ONEWIRE_A: track 49.1 -> 47.0 mm
- net 5V: track 89.4 -> 91.1 mm
- net GPIO_A: track 28.9 -> 29.6 mm
Other:
- board text added: "2.1"
- board text added: "7/2/2013"
- board text removed: "5/8/2013"
